File: scale_heli_leds.sch (KiCad schematic (older format))
At the start: 22 parts, among them IC1 ATTINY85-S, J1 CONN_XH_4POS, J2 HEADER_4POS_2.50mm, P1 pkl_USB_OTG, U1 USBLC6-2, U2 CL320SG-G, U3 MIC5225-3.3V

Commit message: Updated to Rev1.1: Fixed battery connector orientation, fixed incorrect BAT54C schematic symbol pin numbers, removed programming pads.
Parts:
- removed GND1, MISO1, MOSI1, SCK1: POGO_PAD_SMD, pkl_pads:PAD_SMD_R_1x1, symbol POGO_PAD_SMD
- removed RESET1: RESET, pkl_pads:PAD_SMD_R_1x1, symbol POGO_PAD_SMD
- C1, C2, C3, C4: symbol C_Small -> scale_heli_leds-rescue:C_Small
- D1: symbol BAT54C -> scale_heli_leds-rescue:BAT54C
- D2: symbol LED_Small_ALT -> scale_heli_leds-rescue:LED_Small_ALT
- IC1: symbol ATTINY85-S -> scale_heli_leds-rescue:ATTINY85-S
- J1: symbol CONN_HEADER_XH_4POS -> scale_heli_leds-rescue:CONN_HEADER_XH_4POS
- J2: symbol HEADER_4POS_2.50mm -> scale_heli_leds-rescue:HEADER_4POS_2.50mm
- P1: symbol pkl_USB_OTG -> pkl_conn:pkl_USB_OTG
- R1, R2, R3, R4: symbol R_Small -> scale_heli_leds-rescue:R_Small
- U1: symbol USBLC6-2 -> pkl_misc:USBLC6-2
- U2: symbol CL320SG-G -> scale_heli_leds-rescue:CL320SG-G
- U3: symbol MIC5225-3.3V -> scale_heli_leds-rescue:MIC5225-3.3V
Connections:
- wire segments 85 -> 77
- no-connect marks 4 -> 5
Other:
- note added: "Changelist\nV1.1:\n\n1) Change polarity of battery connector\n2) Change DIODE pins BAT54\n3) Dont need ground, need VCC with LED groups - Added VBATT\n4) Removed programming pads\n"
